File: Eagle/EFIS/EFIS.brd (EAGLE design)
At the start: 116.8 x 61.9 mm, 0 parts

Commit message: Initial board layout
Parts:
- added ARPT, DATA, FPV, MTRS, POS, STA, TERR, WPT, WXR: (no value), switch-omron:B3F-10XX
- added BARO, MINS: MERP12246GR, encoder:MERP1224126
- added MODE, RANGE: (no value), switch:CK101X12
- added S1, S2: (no value), switch-custom:320-916
- added T1, T2: (no value), con-lsta:FE15
Changed lines of the file:
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@@
 <layer number="47" name="Measures" color="7" fill="1" visible="no" active="yes"/>
 <layer number="48" name="Document" color="7" fill="1" visible="yes" active="yes"/>
-<layer number="49" name="Reference" color="7" fill="1" visible="yes" active="yes"/>
+<layer number="49" name="Reference" color="7" fill="1" visible="no" active="yes"/>
 <layer number="51" name="tDocu" color="7" fill="1" visible="yes" active="yes"/>
 <layer number="52" name="bDocu" color="7" fill="1" visible="yes" active="yes"/>
@@
 <hole x="112.8903" y="56.9595" drill="3.0734"/>
 <hole x="112.8903" y="4.5212" drill="3.0734"/>
-<circle x="23.5966" y="42.9006" radius="5.08" width="0.4064" layer="25"/>
-<circle x="93.2434" y="42.9006" radius="5.08" width="0.4064" layer="25"/>
-<circle x="47.9552" y="48.9712" radius="4.826" width="0.4064" layer="25"/>
-<circle x="68.58" y="48.9712" radius="4.826" width="0.4064" layer="25"/>
-<circle x="43.1038" y="23.7236" radius="4.826" width="0.4064" layer="25"/>
-<circle x="73.3552" y="23.7236" radius="4.826" width="0.4064" layer="25"/>
-<rectangle x1="8.89" y1="21.59" x2="11.43" y2="29.21" layer="25"/>
-<rectangle x1="105.029" y1="21.59" x2="107.569" y2="29.21" layer="25"/>
-<rectangle x1="8.128" y1="2.7432" x2="18.6436" y2="13.2588" layer="25"/>
-<rectangle x1="23.1648" y1="2.7432" x2="33.782" y2="13.2588" layer="25"/>
-<rectangle x1="38.1508" y1="2.7432" x2="48.7934" y2="13.2588" layer="25"/>
-<rectangle x1="53.1368" y1="2.7432" x2="63.6778" y2="13.2588" layer="25"/>
-<rectangle x1="68.1228" y1="2.7432" x2="78.6638" y2="13.2588" layer="25"/>
-<rectangle x1="83.1596" y1="2.7432" x2="93.5736" y2="13.2588" layer="25"/>
-<rectangle x1="98.171" y1="2.7432" x2="108.6866" y2="13.2588" layer="25"/>
+<circle x="23.5966" y="42.9006" radius="5.08" width="0.4064" layer="49"/>
+<circle x="93.2434" y="42.9006" radius="5.08" width="0.4064" layer="49"/>
+<circle x="47.9552" y="48.9712" radius="4.826" width="0.4064" layer="49"/>
+<circle x="68.58" y="48.9712" radius="4.826" width="0.4064" layer="49"/>
+<circle x="43.1038" y="23.7236" radius="4.826" width="0.4064" layer="49"/>
+<circle x="73.3552" y="23.7236" radius="4.826" width="0.4064" layer="49"/>
+<rectangle x1="8.89" y1="21.59" x2="11.43" y2="29.21" layer="49"/>
+<rectangle x1="105.029" y1="21.59" x2="107.569" y2="29.21" layer="49"/>
+<rectangle x1="8.128" y1="2.7432" x2="18.6436" y2="13.2588" layer="49"/>
+<rectangle x1="23.1648" y1="2.7432" x2="33.782" y2="13.2588" layer="49"/>
+<rectangle x1="38.1508" y1="2.7432" x2="48.7934" y2="13.2588" layer="49"/>
+<rectangle x1="53.1368" y1="2.7432" x2="63.6778" y2="13.2588" layer="49"/>
+<rectangle x1="68.1228" y1="2.7432" x2="78.6638" y2="13.2588" layer="49"/>
+<rectangle x1="83.1596" y1="2.7432" x2="93.5736" y2="13.2588" layer="49"/>
+<rectangle x1="98.171" y1="2.7432" x2="108.6866" y2="13.2588" layer="49"/>
 </plain>
 <attributes>
@@
 </autorouter>
 <elements>
+<element name="T2" library="con-lsta" package="FE15" value="" x="58.42" y="57.15">
+<attribute name="OC_NEWARK" value="unknown" x="58.42" y="57.15" size="1.778" layer="27" display="off"/>
+<attribute name="MPN" value="" x="58.42" y="57.15" size="1.778" layer="27" display="off"/>
+<attribute name="MF" value="" x="58.42" y="57.15" size="1.778" layer="27" display="off"/>
+<attribute name="OC_FARNELL" value="unknown" x="58.42" y="57.15" size="1.778" layer="27" display="off"/>
+</element>
+<element name="T1" library="con-lsta" package="FE15" value="" x="58.42" y="41.91">
+<attribute name="OC_NEWARK" value="unknown" x="58.42" y="41.91" size="1.778" layer="27" display="off"/>
+<attribute name="MPN" value="" x="58.42" y="41.91" size="1.778" layer="27" display="off"/>
+<attribute name="MF" value="" x="58.42" y="41.91" size="1.778" layer="27" display="off"/>
+<attribute name="OC_FARNELL" value="unknown" x="58.42" y="41.91" size="1.778" layer="27" display="off"/>
+</element>
+<element name="FPV" library="switch-omron" package="B3F-10XX" value="" x="48.006" y="49.149">
+<attribute name="OC_NEWARK" value="36M3542" x="48.006" y="49.149" size="1.778" layer="27" display="off"/>
+<attribute name="MPN" value="B3F-1000" x="48.006" y="49.149" size="1.778" layer="27" display="off"/>
+<attribute name="MF" value="" x="48.006" y="49.149" size="1.778" layer="27" display="off"/>
+<attribute name="OC_FARNELL" value="176432" x="48.006" y="49.149" size="1.778" layer="27" display="off"/>
+</element>
+<element name="MTRS" library="switch-omron" package="B3F-10XX" value="" x="68.58" y="49.149">
+<attribute name="OC_NEWARK" value="36M3542" x="68.58" y="49.149" size="1.778" layer="27" display="off"/>
+<attribute name="MPN" value="B3F-1000" x="68.58" y="49.149" size="1.778" layer="27" display="off"/>
+<attribute name="MF" value="" x="68.58" y="49.149" size="1.778" layer="27" display="off"/>
+<attribute name="OC_FARNELL" value="176432" x="68.58" y="49.149" size="1.778" layer="27" display="off"/>
+</element>
+<element name="WXR" library="switch-omron" package="B3F-10XX" value="" x="13.335" y="7.62">
+<attribute name="OC_NEWARK" value="36M3542" x="13.335" y="7.62" size="1.778" layer="27" display="off"/>
+<attribute name="MPN" value="B3F-1000" x="13.335" y="7.62" size="1.778" layer="27" display="off"/>
+<attribute name="MF" value="" x="13.335" y="7.62" size="1.778" layer="27" display="off"/>
+<attribute name="OC_FARNELL" value="176432" x="13.335" y="7.62" size="1.778" layer="27" display="off"/>
+</element>
+<element name="STA" library="switch-omron" package="B3F-10XX" value="" x="28.575" y="7.62">
+<attribute name="OC_NEWARK" value="36M3542" x="28.575" y="7.62" size="1.778" layer="27" display="off"/>
+<attribute name="MPN" value="B3F-1000" x="28.575" y="7.62" size="1.778" layer="27" display="off"/>
+<attribute name="MF" value="" x="28.575" y="7.62" size="1.778" layer="27" display="off"/>
+<attribute name="OC_FARNELL" value="176432" x="28.575" y="7.62" size="1.778" layer="27" display="off"/>
+</element>
+<element name="WPT" library="switch-omron" package="B3F-10XX" value="" x="43.4975" y="7.62">
+<attribute name="OC_NEWARK" value="36M3542" x="43.4975" y="7.62" size="1.778" layer="27" display="off"/>
+<attribute name="MPN" value="B3F-1000" x="43.4975" y="7.62" size="1.778" layer="27" display="off"/>
+<attribute name="MF" value="" x="43.4975" y="7.62" size="1.778" layer="27" display="off"/>
+<attribute name="OC_FARNELL" value="176432" x="43.4975" y="7.62" size="1.778" layer="27" display="off"/>
+</element>
+<element name="ARPT" library="switch-omron" package="B3F-10XX" value="" x="58.42" y="7.62">
+<attribute name="OC_NEWARK" value="36M3542" x="58.42" y="7.62" size="1.778" layer="27" display="off"/>
+<attribute name="MPN" value="B3F-1000" x="58.42" y="7.62" size="1.778" layer="27" display="off"/>
+<attribute name="MF" value="" x="58.42" y="7.62" size="1.778" layer="27" display="off"/>
+<attribute name="OC_FARNELL" value="176432" x="58.42" y="7.62" size="1.778" layer="27" display="off"/>
+</element>
+<element name="DATA" library="switch-omron" package="B3F-10XX" value="" x="73.3425" y="7.62">
+<attribute name="OC_NEWARK" value="36M3542" x="73.3425" y="7.62" size="1.778" layer="27" display="off"/>
+<attribute name="MPN" value="B3F-1000" x="73.3425" y="7.62" size="1.778" layer="27" display="off"/>
+<attribute name="MF" value="" x="73.3425" y="7.62" size="1.778" layer="27" display="off"/>
+<attribute name="OC_FARNELL" value="176432" x="73.3425" y="7.62" size="1.778" layer="27" display="off"/>
+</element>
+<element name="POS" library="switch-omron" package="B3F-10XX" value="" x="88.392" y="7.62">
+<attribute name="OC_NEWARK" value="36M3542" x="88.392" y="7.62" size="1.778" layer="27" display="off"/>
+<attribute name="MPN" value="B3F-1000" x="88.392" y="7.62" size="1.778" layer="27" display="off"/>
+<attribute name="MF" value="" x="88.392" y="7.62" size="1.778" layer="27" display="off"/>
+<attribute name="OC_FARNELL" value="176432" x="88.392" y="7.62" size="1.778" layer="27" display="off"/>
+</element>
+<element name="TERR" library="switch-omron" package="B3F-10XX" value="" x="103.505" y="7.62">
+<attribute name="OC_NEWARK" value="36M3542" x="103.505" y="7.62" size="1.778" layer="27" display="off"/>
+<attribute name="MPN" value="B3F-1000" x="103.505" y="7.62" size="1.778" layer="27" display="off"/>
+<attribute name="MF" value="" x="103.505" y="7.62" size="1.778" layer="27" display="off"/>
+<attribute name="OC_FARNELL" value="176432" x="103.505" y="7.62" size="1.778" layer="27" display="off"/>
+</element>
+<element name="MODE" library="switch" package="CK101X12" value="" x="43.1038" y="23.749" rot="R180"/>
+<element name="RANGE" library="switch" package="CK101X12" value="" x="73.3552" y="23.749" rot="R180"/>
+<element name="MINS" library="encoder" package="MERP1224126" value="MERP12246GR" x="90.7034" y="35.433"/>
+<element name="BARO" library="encoder" package="MERP1224126" value="MERP12246GR" x="21.0185" y="35.433"/>
+<element name="S1" library="switch-custom" package="320-916" value="" x="10.19175" y="25.4"/>
+<element name="S2" library="switch-custom" package="320-916" value="" x="106.299" y="25.4"/>
 </elements>
 <signals>

Commit message: Button connections in Eagle
Parts:
- added C1, C10, C11, C12, C13, C2, C3, C4, C5, C6, C7, C8, C9: 100nF, rcl:C1206
- added R1, R10, R11, R12, R13, R2, R3, R4, R5, R6, R7, R8, R9: 10K, resistor:R1206
- renumbered S1 to VOR1, S2 to VOR2
Connections:
- new net ARPT: ARPT.2, C4.1, T2.10
- new net DATA: C5.1, DATA.2, T2.11
- new net GND: R1.2, R10.1, R11.1, R12.2, R13.2, R2.2, R3.2, R4.2, R5.2, R6.2, R7.2, R8.1, R9.1, T2.1
- new net N$1: R1.1, WXR.1
- new net N$10: POS.1, R6.1
- new net N$11: R7.1, TERR.1
- new net N$12: FPV.1, R12.1
- new net N$13: MTRS.1, R13.1
- new net N$14: C12.1, FPV.2, T1.4
- new net N$15: C13.1, MTRS.2, T1.5
- new net N$2: C8.2, R8.2, T2.3, VOR1.1
- new net N$3: C9.2, R9.2, T2.4, VOR1.3
- new net N$4: R2.1, STA.1
- new net N$5: R3.1, WPT.1
- new net N$6: C10.2, R10.2, T2.5, VOR2.1
- new net N$7: C11.2, R11.2, T2.6, VOR2.3
- new net N$8: ARPT.1, R4.1
- new net N$9: DATA.1, R5.1
- new net POS: C6.1, POS.2, T2.12
- new net STA: C2.1, STA.2, T2.8
- new net TERR: C7.1, T2.13, TERR.2
- new net VCC: ARPT.4, C1.2, C10.1, C11.1, C12.2, C13.2, C2.2, C3.2, C4.2, C5.2, C6.2, C7.2, C8.1, C9.1, DATA.4, FPV.4, MTRS.4, POS.4, STA.4, T1.3, TERR.4, VOR1.2, VOR2.2, WPT.4, WXR.4
- new net WPT: C3.1, T2.9, WPT.2
- new net WXR: C1.1, T2.7, WXR.2
Routing:
- net VCC: track 0.00 -> 325.8 mm, vias 0 -> 1
- net WXR: track 0.00 -> 112.6 mm
- net N$7: track 0.00 -> 92.6 mm, vias 0 -> 1
- net N$3: track 0.00 -> 86.6 mm
- net N$6: track 0.00 -> 85.4 mm, vias 0 -> 1
- net TERR: track 0.00 -> 78.3 mm, vias 0 -> 1
- net N$2: track 0.00 -> 77.4 mm
- net POS: track 0.00 -> 72.9 mm, vias 0 -> 1
- net DATA: track 0.00 -> 71.3 mm
- net ARPT: track 0.00 -> 69.7 mm
- net STA: track 0.00 -> 66.9 mm
- net WPT: track 0.00 -> 60.1 mm, vias 0 -> 1
- net N$15: track 0.00 -> 39.3 mm
- net N$14: track 0.00 -> 17.3 mm
- net N$11: track 0.00 -> 12.5 mm
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- added copper zone on layer 16, net GND

Commit message: All components placed and some manual routing
Parts:
- added R14, R19: 5.1K, resistor:R1206
- added R15, R20: 10K, resistor:R1206
- added R16, R21: 15K, resistor:R1206
- added R17, R22: 20K, resistor:R1206
- added R18, R27: 100K, resistor:R1206
- added R23: 24K, resistor:R1206
- added R24: 30K, resistor:R1206
- added R25: 36K, resistor:R1206
- added R26: 47K, resistor:R1206
- moved BARO 69.7 mm to (90.7, 35.4)
- moved MINS 69.7 mm to (21.0, 35.4)
- moved R2 0.32 mm to (28.9, 2.54)
- moved C7 0.32 mm to (111.8, 9.84), turned to 180 degrees
- moved R1 0.32 mm to (5.08, 9.84)
- turned C11 to 90 degrees
- turned C9 to 90 degrees
Connections:
- net N$14 renamed FPV
- net N$15 renamed MTRS
- net N$2 renamed VOR1
- net N$6 renamed VOR2
- removed net N$3: C9.2, R9.2, T2.4, VOR1.3
- removed net N$7: C11.2, R11.2, T2.6, VOR2.3
- new net ADF1: C9.1, R9.2, T2.4, VOR1.3
- new net ADF2: C11.1, R11.2, T2.6, VOR2.3
- new net BAROA: BARO.A, T1.8
- new net BAROB: BARO.B, T1.9
- new net BAROSTD: BARO.4, T1.11
- new net LED1: MINS.2, T1.14
- new net MINSA: MINS.A, T1.6
- new net MINSB: MINS.B, T1.7
- new net MINSRST: MINS.4, T1.10
- new net MODE: R14.1, R15.1, R16.1, R17.1, R18.2, T1.13
- new net N$16: MODE.1, R14.2
- new net N$17: MODE.2, R15.2
- new net N$18: MODE.3, R16.2
- new net N$19: MODE.4, R17.2
- new net N$21: R19.2, RANGE.1
- new net N$22: R20.2, RANGE.2
- new net N$23: R21.2, RANGE.3
- new net N$24: R22.2, RANGE.4
- new net N$25: R23.2, RANGE.5
- new net N$26: R24.2, RANGE.6
- new net N$27: R25.2, RANGE.7
- new net N$28: R26.2, RANGE.8
- new net RANGE: R19.1, R20.1, R21.1, R22.1, R23.1, R24.1, R25.1, R26.1, R27.2, T1.12
- net GND: now also BARO.1, BARO.C, MINS.1, MINS.C, R18.1, R27.1, T1.2
- net VCC: now also C11.2, C9.2, MODE.A, RANGE.A; no longer C11.1, C9.1
Routing:
- net N$7: track 92.6 -> 0.00 mm, vias 1 -> 0
- net N$3: track 86.6 -> 0.00 mm
- net TERR: track 78.3 -> 3.60 mm, vias 1 -> 0
- net VOR2: track 85.4 -> 14.0 mm, vias 1 -> 0
- net POS: track 72.9 -> 3.71 mm, vias 1 -> 0
- net DATA: track 71.3 -> 3.52 mm
- net ARPT: track 69.7 -> 3.22 mm
- net ADF1: track 0.00 -> 66.0 mm
- net STA: track 66.9 -> 3.22 mm
- net WPT: track 60.1 -> 3.52 mm, vias 1 -> 0
- net MINSRST: track 0.00 -> 48.5 mm
- net MINSA: track 0.00 -> 39.9 mm
- net BAROB: track 0.00 -> 39.2 mm
- net WXR: track 112.6 -> 75.3 mm
- net BAROA: track 0.00 -> 37.1 mm
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
Commit message: REV 1 PCB
Parts:
- moved T1 15.2 mm to (58.4, 57.1)
- moved T2 15.2 mm to (58.4, 41.9)
Connections:
- net MODE: now also T1.12; no longer T1.13
- net RANGE: now also T1.13; no longer T1.12
Routing:
- net RANGE: track 0.00 -> 95.2 mm, vias 0 -> 1
- net ADF2: track 14.0 -> 77.8 mm, vias 0 -> 1
- net VOR2: track 14.0 -> 76.2 mm
- net TERR: track 3.60 -> 65.5 mm
- net LED1: track 0.00 -> 57.1 mm
- net MODE: track 0.00 -> 52.0 mm, vias 0 -> 1
- net STA: track 3.22 -> 45.9 mm, vias 0 -> 1
- net POS: track 3.71 -> 45.9 mm, vias 0 -> 1
- net WPT: track 3.52 -> 44.0 mm
- net DATA: track 3.52 -> 40.6 mm
- net ARPT: track 3.22 -> 38.8 mm
- net MTRS: track 4.85 -> 35.8 mm
- net MINSB: track 36.9 -> 58.5 mm
- net VCC: track 318.6 -> 338.2 mm, vias 4 -> 0
- net WXR: track 75.3 -> 56.4 mm, vias 0 -> 1
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Other:
- board text added: "B737 EFIS PANEL REV 1"
